Commit message: use diff_drive_controller

File: vagrant_description/model/motor.urdf.xacro (robot description, xacro)
@@ -14,8 +14,8 @@
 <robot xmlns:xacro="http://www.ros.org/wiki/xacro" name="motor">
     <xacro:include filename="$(find urdf_juggle)/inertials.urdf.xacro" />
-    <xacro:macro name="wheel_motor" params="name">
-        <xacro:property name="stator_name" value="${name}_stator" scope="global"/>
+    <xacro:macro name="wheel_motor" params="name base xyz rpy">
+        <xacro:property name="stator_name" value="${name}_stator" />
         <xacro:property name="rotor_name" value="${name}_rotor" />
-        <xacro:property name="joint_name" value="${name}_joint_stator_to_rotor" />
+        <xacro:property name="joint_name" value="${name}_joint_base_to_rotor" />
     	<link name="${stator_name}">
     		<visual>
@@ -42,8 +42,8 @@
     		</inertial>
     	</link>
-    	<joint name="${joint_name}" type="continuous">
-    		<parent link="${stator_name}" />
-    		<child link="${rotor_name}" />
-            <dynamics friction="0.024" />
+    	<joint name="${name}_base_to_stator" type="fixed">
+    	   <parent link="${base}" />
+    	   <child link="${stator_name}" />
+    	   <origin xyz="${xyz}" rpy="${rpy}" />
     	</joint>
     	<link name="${rotor_name}">
@@ -75,11 +75,17 @@
             <kd>0.2</kd>
         </gazebo>
+        <joint name="${joint_name}" type="continuous">
+            <parent link="${base}" />
+            <child link="${rotor_name}" />
+            <dynamics friction="0.024" />
+            <origin xyz="${xyz}" rpy="${rpy}" />
+        </joint>
     	<transmission name="${name}_rotor_transmission">
     		<type>transmission_interface/SimpleTransmission</type>
     		<joint name="${joint_name}">
-    			<hardwareInterface>hardware_interface/EffortJointInterface</hardwareInterface>
+    			<hardwareInterface>hardware_interface/VelocityJointInterface</hardwareInterface>
     		</joint>
     		<actuator name="${name}_motor">
-    			<hardwareInterface>hardware_interface/EffortJointInterface</hardwareInterface>
+    			<hardwareInterface>hardware_interface/VelocityJointInterface</hardwareInterface>
     			<mechanicalReduction>171</mechanicalReduction>
     		</actuator>

File: vagrant_description/model/vagrant.urdf.xacro (robot description, xacro)
@@ -45,10 +45,5 @@
     <xacro:include filename="$(find vagrant_description)/model/motor.urdf.xacro" />
     <xacro:macro name="robot_motor" params="name x y yaw">
-        <xacro:wheel_motor name="${name}" />
-        <joint name="body_to_${name}" type="fixed">
-            <parent link="body" />
-            <child link="${stator_name}" />
-            <origin xyz="${x} ${y} -0.022" rpy="0.0 0.0 ${yaw}" />
-        </joint>
+        <xacro:wheel_motor name="${name}" base="base_link" xyz="${x} ${y} -0.022" rpy="0.0 0.0 ${yaw}" />
     </xacro:macro>
     <xacro:robot_motor name="left_front_motor" x="0.0635" y="0.095" yaw="1.571" />

Commit message: adjust model physics

File: vagrant_description/model/motor.urdf.xacro (robot description, xacro)
@@ -18,77 +18,78 @@
         <xacro:property name="rotor_name" value="${name}_rotor" />
         <xacro:property name="joint_name" value="${name}_joint_base_to_rotor" />
-    	<link name="${stator_name}">
-    		<visual>
-    			<geometry>
-    				<mesh filename="file://$(find vagrant_description)/model/wheel_motor_stator/wheel_motor_stator.dae" />
-    			</geometry>
-    			<origin xyz="-0.0205 0 0" />
-    		</visual>
-    		<collision>
-    			<geometry>
-    				<box size="0.0645 0.026 0.024" />
-    			</geometry>
-    			<origin xyz="-0.0535 0.0005 0" />
-    		</collision>
-    		<collision>
-    			<geometry>
-    				<box size="0.033 0.026 0.01" />
-    			</geometry>
-    			<origin xyz="-0.037 0 0.017"/>
-    		</collision>
-    		<inertial>
-    			<origin xyz="-0.048 0 0.003" />
-    			<xacro:box_inertia mass="0.1" size="0.064 0.024 0.03" />
-    		</inertial>
-    	</link>
-    	<joint name="${name}_base_to_stator" type="fixed">
-    	   <parent link="${base}" />
-    	   <child link="${stator_name}" />
-    	   <origin xyz="${xyz}" rpy="${rpy}" />
-    	</joint>
-    	<link name="${rotor_name}">
-    		<visual>
-    			<geometry>
-    				<mesh filename="file://$(find vagrant_description)/model/wheel_motor_rotor/wheel_motor_rotor.dae" />
-    			</geometry>
-    		</visual>
-    		<collision>
-    			<geometry>
-    				<cylinder radius="0.0337" length="0.025" />
-    			</geometry>
-    			<origin xyz="-0.0002 0 0" rpy="0 1.571 0" />
-    		</collision>
-    		<collision>
-    			<geometry>
-    				<cylinder radius="0.0055" length="0.0072" />
-    			</geometry>
-    			<origin xyz="-0.0165 0 0" rpy="0 1.571 0" />
-    		</collision>
-    		<inertial>
-    			<xacro:cylinder_inertia mass="0.05" radius="0.032" length="0.028" />
-    			<origin rpy="0 1.571 0" />
-    		</inertial>
-    	</link>
+        <link name="${stator_name}">
+            <visual>
+                <geometry>
+                    <mesh filename="file://$(find vagrant_description)/model/wheel_motor_stator/wheel_motor_stator.dae" />
+                </geometry>
+                <origin xyz="-0.0205 0 0" />
+            </visual>
+            <collision>
+                <geometry>
+                    <box size="0.0645 0.026 0.024" />
+                </geometry>
+                <origin xyz="-0.0535 0.0005 0" />
+            </collision>
+            <collision>
+                <geometry>
+                    <box size="0.033 0.026 0.01" />
+                </geometry>
+                <origin xyz="-0.037 0 0.017"/>
+            </collision>
+            <inertial>
+                <origin xyz="-0.048 0 0.003" />
+                <xacro:box_inertia mass="0.1" size="0.064 0.024 0.03" />
+            </inertial>
+        </link>
+        <joint name="${name}_base_to_stator" type="fixed">
+           <parent link="${base}" />
+           <child link="${stator_name}" />
+           <origin xyz="${xyz}" rpy="${rpy}" />
+        </joint>
+        <link name="${rotor_name}">
+            <visual>
+                <geometry>
+                    <mesh filename="file://$(find vagrant_description)/model/wheel_motor_rotor/wheel_motor_rotor.dae" />
+                </geometry>
+            </visual>
+            <collision>
+                <geometry>
+                    <cylinder radius="0.0337" length="0.025" />
+                </geometry>
+                <origin xyz="-0.0002 0 0" rpy="0 1.571 0" />
+            </collision>
+            <collision>
+                <geometry>
+                    <cylinder radius="0.0055" length="0.0072" />
+                </geometry>
+                <origin xyz="-0.0165 0 0" rpy="0 1.571 0" />
+            </collision>
+            <inertial>
+                <xacro:cylinder_inertia mass="0.05" radius="0.032" length="0.028" />
+                <origin rpy="0 1.571 0" />
+            </inertial>
+        </link>
         <gazebo reference="${rotor_name}">
             <mu1>0.8</mu1>
             <mu2>0.8</mu2>
-            <kd>0.2</kd>
+            <kp>8.0e+3</kp>
+            <kd>100.0</kd>
         </gazebo>
         <joint name="${joint_name}" type="continuous">
             <parent link="${base}" />
             <child link="${rotor_name}" />
-            <dynamics friction="0.024" />
+            <dynamics friction="0.031" />
             <origin xyz="${xyz}" rpy="${rpy}" />
         </joint>
-    	<transmission name="${name}_rotor_transmission">
-    		<type>transmission_interface/SimpleTransmission</type>
-    		<joint name="${joint_name}">
-    			<hardwareInterface>hardware_interface/VelocityJointInterface</hardwareInterface>
-    		</joint>
-    		<actuator name="${name}_motor">
-    			<hardwareInterface>hardware_interface/VelocityJointInterface</hardwareInterface>
-    			<mechanicalReduction>171</mechanicalReduction>
-    		</actuator>
-    	</transmission>
+        <transmission name="${name}_rotor_transmission">
+            <type>transmission_interface/SimpleTransmission</type>
+            <joint name="${joint_name}">
+                <hardwareInterface>hardware_interface/VelocityJointInterface</hardwareInterface>
+            </joint>
+            <actuator name="${name}_motor">
+                <hardwareInterface>hardware_interface/VelocityJointInterface</hardwareInterface>
+                <mechanicalReduction>1</mechanicalReduction>
+            </actuator>
+        </transmission>
     </xacro:macro>
 </robot>

File: vagrant_description/model/vagrant.urdf.xacro (robot description, xacro)
@@ -36,5 +36,5 @@
         <inertial>
             <xacro:box_inertia mass="2.0" size="0.21 0.22 0.127" />
-            <origin xyz="0.002 0.0 0.064" />
+            <origin xyz="-0.002 0.0 0.064" />
         </inertial>
     </link>
